File: pcb/LeoSDVX-Shield.sch (KiCad schematic (older format))
At the start: 11 parts, among them J1 JST-XH, J10 Conn_01x02, J2 JST-XH, J3 JST-XH, J4 JST-XH, J5 JST-XH, J6 JST-XH, J7 JST-XH, J8 JST-XH, J9 JST-XH

Commit message: Revision 2
REV 2 released

- Replaced JST-XH connector footprints with generic 2.54mm header footprints, original footprints were well out of spec and didn't fit 2.54mm headers/plugs; thank you SirusDoma (C&S discord) for bringing this to my attention.

- System pin rotated to have GND on the same side as all other connections (I have also forgotten why the system pin exists but I'm leaving it there /shrug)

- Removed white border on leonardo shield footprint, library updated and included

Hopefully the last update this will need
Parts:
- removed J1, J2, J3, J4, J5, J6, J7, J8, J9: JST-XH, Connectors:JST-4-PTH-VERT, symbol CONN_04JST-PTH-VERT
- added J1, J2, J3, J4, J5, J6, J7, J8, J9: CONN_04, Pin_Headers:Pin_Header_Straight_1x04_Pitch2.54mm, symbol CONN_04
- XA1: footprint Arduino:Arduino_Leonardo_Shield -> Arduino:Arduino_Leonardo_Shield_noborder
Connections:
- net B1: now also J3.3
- net B1LED: now also J3.4
- net B2: now also J4.3
- net B2LED: now also J4.4
- net B3: now also J5.3
- net B3LED: now also J5.4
- net B4: now also J6.3
- net B4LED: now also J6.4
- net B5: now also J7.3
- net B5LED: now also J7.4
- net B6: now also J8.3
- net B6LED: now also J8.4
- net B7: now also J9.3
- net B7LED: now also J9.4
- net E1D+: now also J1.4
- net E1D-: now also J1.3
- net E2D+: now also J2.4
- net E2D-: now also J2.3
- net GND: now also J1.1, J2.1, J3.1, J3.2, J4.1, J4.2, J5.1, J5.2, J6.1, J6.2, J7.1, J7.2, J8.1, J8.2, J9.1, J9.2
- net VCC: now also J1.2, J2.2
Changed lines of the file:
@@
 $EndDescr
-$Comp
-L CONN_04JST-PTH-VERT J3
-U 1 1 5B6C5898
-P 2900 3900
-F 0 "J3" H 2700 4300 45  0000 L BNN
-F 1 "JST-XH" H 2700 3750 45  0000 L BNN
-F 2 "Connectors:JST-4-PTH-VERT" H 2900 4400 20  0001 C CNN
-F 3 "" H 2900 3900 50  0001 C CNN
-F 4 "Button 1" H 2900 4450 60  0000 C CNN "Field4"
-	1    2900 3900
-	0    -1   -1   0
-$EndComp
-$Comp
-L CONN_04JST-PTH-VERT J5
-U 1 1 5B6C58E2
-P 3950 3900
-F 0 "J5" H 3750 4300 45  0000 L BNN
-F 1 "JST-XH" H 3750 3750 45  0000 L BNN
-F 2 "Connectors:JST-4-PTH-VERT" H 3950 4400 20  0001 C CNN
-F 3 "" H 3950 3900 50  0001 C CNN
-F 4 "Button 3" H 3950 4450 60  0000 C CNN "Field4"
-	1    3950 3900
-	0    -1   -1   0
-$EndComp
-$Comp
-L CONN_04JST-PTH-VERT J7
-U 1 1 5B6C5933
-P 5000 3900
-F 0 "J7" H 4800 4300 45  0000 L BNN
-F 1 "JST-XH" H 4800 3750 45  0000 L BNN
-F 2 "Connectors:JST-4-PTH-VERT" H 5000 4400 20  0001 C CNN
-F 3 "" H 5000 3900 50  0001 C CNN
-F 4 "Button 5" H 5000 4450 60  0000 C CNN "Field4"
-	1    5000 3900
-	0    -1   -1   0
-$EndComp
-$Comp
-L CONN_04JST-PTH-VERT J9
-U 1 1 5B6C595B
-P 6050 3900
-F 0 "J9" H 5850 4300 45  0000 L BNN
-F 1 "JST-XH" H 5850 3750 45  0000 L BNN
-F 2 "Connectors:JST-4-PTH-VERT" H 6050 4400 20  0001 C CNN
-F 3 "" H 6050 3900 50  0001 C CNN
-F 4 "Button 7" H 6050 4450 60  0000 C CNN "Field4"
-	1    6050 3900
-	0    -1   -1   0
-$EndComp
-$Comp
-L CONN_04JST-PTH-VERT J4
-U 1 1 5B6C5990
-P 3350 4700
-F 0 "J4" H 3150 5100 45  0000 L BNN
-F 1 "JST-XH" H 3150 4550 45  0000 L BNN
-F 2 "Connectors:JST-4-PTH-VERT" H 3350 5200 20  0001 C CNN
-F 3 "" H 3350 4700 50  0001 C CNN
-F 4 "Button 2" H 3350 5250 60  0000 C CNN "Field4"
-	1    3350 4700
-	0    -1   -1   0
-$EndComp
-$Comp
-L CONN_04JST-PTH-VERT J6
-U 1 1 5B6C59CA
-P 4400 4700
-F 0 "J6" H 4200 5100 45  0000 L BNN
-F 1 "JST-XH" H 4200 4550 45  0000 L BNN
-F 2 "Connectors:JST-4-PTH-VERT" H 4400 5200 20  0001 C CNN
-F 3 "" H 4400 4700 50  0001 C CNN
-F 4 "Button 4" H 4400 5250 60  0000 C CNN "Field4"
-	1    4400 4700
-	0    -1   -1   0
-$EndComp
-$Comp
-L CONN_04JST-PTH-VERT J8
-U 1 1 5B6C5A05
-P 5450 4700
-F 0 "J8" H 5250 5100 45  0000 L BNN
-F 1 "JST-XH" H 5250 4550 45  0000 L BNN
-F 2 "Connectors:JST-4-PTH-VERT" H 5450 5200 20  0001 C CNN
-F 3 "" H 5450 4700 50  0001 C CNN
-F 4 "Button 6" H 5450 5250 60  0000 C CNN "Field4"
-	1    5450 4700
-	0    -1   -1   0
-$EndComp
-$Comp
-L CONN_04JST-PTH-VERT J2
-U 1 1 5B6C65BF
-P 2300 4700
-F 0 "J2" H 2100 5100 45  0000 L BNN
-F 1 "JST-XH" H 2100 4550 45  0000 L BNN
-F 2 "Connectors:JST-4-PTH-VERT" H 2300 5200 20  0001 C CNN
-F 3 "" H 2300 4700 50  0001 C CNN
-F 4 "Encoder 2" H 2300 5250 60  0000 C CNN "Field4"
-	1    2300 4700
-	0    -1   -1   0
-$EndComp
-$Comp
-L CONN_04JST-PTH-VERT J1
-U 1 1 5B6C65F9
-P 1850 3900
-F 0 "J1" H 1650 4300 45  0000 L BNN
-F 1 "JST-XH" H 1650 3750 45  0000 L BNN
-F 2 "Connectors:JST-4-PTH-VERT" H 1850 4400 20  0001 C CNN
-F 3 "" H 1850 3900 50  0001 C CNN
-F 4 "Encoder 1" H 1850 4450 60  0000 C CNN "Field4"
-	1    1850 3900
-	0    -1   -1   0
-$EndComp
 $Comp
 L Arduino_Leonardo_Shield XA1
@@
 F 0 "XA1" V 8500 2350 60  0000 C CNN
 F 1 "Arduino_Leonardo_Shield" V 8300 2350 60  0000 C CNN
-F 2 "Arduino:Arduino_Leonardo_Shield" H 10200 6100 60  0001 C CNN
+F 2 "Arduino:Arduino_Leonardo_Shield_noborder" H 10200 6100 60  0001 C CNN
 F 3 "" H 10200 6100 60  0001 C CNN
 	1    8400 2350
@@
 Wire Wire Line
 	10150 1600 9700 1600
+$Comp
+L CONN_04 J9
+U 1 1 5CCFC5BB
+P 6050 3900
+F 0 "J9" H 5850 4300 45  0000 L BNN
+F 1 "CONN_04" H 5850 3750 45  0000 L BNN
+F 2 "Pin_Headers:Pin_Header_Straight_1x04_Pitch2.54mm" H 6050 4400 20  0001 C CNN
+F 3 "" H 6050 3900 50  0001 C CNN
+F 4 "Button 7" H 6050 4450 60  0000 C CNN "Field4"
+	1    6050 3900
+	0    -1   -1   0
+$EndComp
+$Comp
+L CONN_04 J7
+U 1 1 5CCFCBBB
+P 5000 3900
+F 0 "J7" H 4800 4300 45  0000 L BNN
+F 1 "CONN_04" H 4800 3750 45  0000 L BNN
+F 2 "Pin_Headers:Pin_Header_Straight_1x04_Pitch2.54mm" H 5000 4400 20  0001 C CNN
+F 3 "" H 5000 3900 50  0001 C CNN
+F 4 "Button 5" H 5000 4450 60  0000 C CNN "Field4"
+	1    5000 3900
+	0    -1   -1   0
+$EndComp
+$Comp
+L CONN_04 J5
+U 1 1 5CCFCC05
+P 3950 3900
+F 0 "J5" H 3750 4300 45  0000 L BNN
+F 1 "CONN_04" H 3750 3750 45  0000 L BNN
+F 2 "Pin_Headers:Pin_Header_Straight_1x04_Pitch2.54mm" H 3950 4400 20  0001 C CNN
+F 3 "" H 3950 3900 50  0001 C CNN
+F 4 "Button 3" H 3950 4450 60  0000 C CNN "Field4"
+	1    3950 3900
+	0    -1   -1   0
+$EndComp
+$Comp
+L CONN_04 J3
+U 1 1 5CCFCC52
+P 2900 3900
+F 0 "J3" H 2700 4300 45  0000 L BNN
+F 1 "CONN_04" H 2700 3750 45  0000 L BNN
+F 2 "Pin_Headers:Pin_Header_Straight_1x04_Pitch2.54mm" H 2900 4400 20  0001 C CNN
+F 3 "" H 2900 3900 50  0001 C CNN
+F 4 "Button 1" H 2900 4450 60  0000 C CNN "Field4"
+	1    2900 3900
+	0    -1   -1   0
+$EndComp
+$Comp
+L CONN_04 J1
+U 1 1 5CCFCCB0
+P 1850 3900
+F 0 "J1" H 1650 4300 45  0000 L BNN
+F 1 "CONN_04" H 1650 3750 45  0000 L BNN
+F 2 "Pin_Headers:Pin_Header_Straight_1x04_Pitch2.54mm" H 1850 4400 20  0001 C CNN
+F 3 "" H 1850 3900 50  0001 C CNN
+F 4 "Encoder 1" H 1850 4450 60  0000 C CNN "Field4"
+	1    1850 3900
+	0    -1   -1   0
+$EndComp
+$Comp
+L CONN_04 J2
+U 1 1 5CCFCD05
+P 2300 4700
+F 0 "J2" H 2100 5100 45  0000 L BNN
+F 1 "CONN_04" H 2100 4550 45  0000 L BNN
+F 2 "Pin_Headers:Pin_Header_Straight_1x04_Pitch2.54mm" H 2300 5200 20  0001 C CNN
+F 3 "" H 2300 4700 50  0001 C CNN
+F 4 "Encoder 2" H 2300 5250 60  0000 C CNN "Field4"
+	1    2300 4700
+	0    -1   -1   0
+$EndComp
+$Comp
+L CONN_04 J4
+U 1 1 5CCFCD57
+P 3350 4700
+F 0 "J4" H 3150 5100 45  0000 L BNN
+F 1 "CONN_04" H 3150 4550 45  0000 L BNN
+F 2 "Pin_Headers:Pin_Header_Straight_1x04_Pitch2.54mm" H 3350 5200 20  0001 C CNN
+F 3 "" H 3350 4700 50  0001 C CNN
+F 4 "Button 2" H 3350 5250 60  0000 C CNN "Field4"
+	1    3350 4700
+	0    -1   -1   0
+$EndComp
+$Comp
+L CONN_04 J6
+U 1 1 5CCFCDB2
+P 4400 4700
+F 0 "J6" H 4200 5100 45  0000 L BNN
+F 1 "CONN_04" H 4200 4550 45  0000 L BNN
+F 2 "Pin_Headers:Pin_Header_Straight_1x04_Pitch2.54mm" H 4400 5200 20  0001 C CNN
+F 3 "" H 4400 4700 50  0001 C CNN
+F 4 "Button 4" H 4400 5250 60  0000 C CNN "Field4"
+	1    4400 4700
+	0    -1   -1   0
+$EndComp
+$Comp
+L CONN_04 J8
+U 1 1 5CCFCE3E
+P 5450 4700
+F 0 "J8" H 5250 5100 45  0000 L BNN
+F 1 "CONN_04" H 5250 4550 45  0000 L BNN
+F 2 "Pin_Headers:Pin_Header_Straight_1x04_Pitch2.54mm" H 5450 5200 20  0001 C CNN
+F 3 "" H 5450 4700 50  0001 C CNN
+F 4 "Button 6" H 5450 5250 60  0000 C CNN "Field4"
+	1    5450 4700
+	0    -1   -1   0
+$EndComp
 $EndSCHEMATC
